File: 05-Layout/nowae020/nowae020-0/nowae020.sch (KiCad schematic (older format))
At the start: 67 parts, among them J1 SMALL_JUMPER, J2 SMALL_JUMPER, J3 SMALL_JUMPER, P1 USB_A_90, Q1 IRLML6402, U1 FT230XQ, U2 TPS62152, U3 BGM111A256V2

Commit message: WiP: schematic (nowae020-0)
Parts:
- removed DL10, DL7, DL8, DL9: GREEN, LEDs:LED-0402, symbol nowae-led:GREEN
- removed DL11, DL12, DL13, DL14, DL15, DL16, DL17: YELLOW, LEDs:LED-0402, symbol nowae-led:YELLOW
- removed DL5: RED, LEDs:LED-0402, symbol nowae-led:RED
- removed DL6: BLUE, LEDs:LED-0402, symbol nowae-led:BLUE
- removed J1, J2, J3: SMALL_JUMPER, MISC:JUMPERSMD-2, symbol nowae-misc:JUMPER-2
- removed R10, R11, R12, R13, R14: 680, RESISTOR:RESISTOR-0402, symbol nowae-resistor:RESISTOR
- removed R15, R16, R17, R18, R19, R20, R21, R9: 1k5, RESISTOR:RESISTOR-0402, symbol nowae-resistor:RESISTOR
- removed R22: 4k7, RESISTOR:RESISTOR-0402, symbol nowae-resistor:RESISTOR
- added C? (x2): 100n, symbol nowae-capacitor:CAPACITOR
- added DL?: GREEN, LEDs:LED-0402, symbol nowae-led:GREEN
- added DL?: BLUE, LEDs:LED-0402, symbol nowae-led:BLUE
- added P? (x3): CONN_8X1, symbol nowae-connector:CONN_8X1
- added R? (x4): 10k, RESISTOR:RESISTOR-0402, symbol nowae-resistor:RESISTOR
- added R? (x2): 287, RESISTOR:RESISTOR-0402, symbol nowae-resistor:RESISTOR
- added SW?: SWITCH1, BUTTON:BUTTON-WE-434153017835, symbol nowae-switch:BUTTON-WE_434153017835
- added SW?: SWITCH0, BUTTON:BUTTON-WE-434153017835, symbol nowae-switch:BUTTON-WE_434153017835
Connections:
- net labels added: LED0, LED1, SWITCH0, SWITCH1
- net labels removed: BATTERY_IND, LINK_DROP, MODE, ON/OFF, P1_2, P1_3, P2_4, P3_5, PAIRING_KEY, PWM1, PWM2, RESET, RSSI_IND, STATUS1_IND, STATUS2_IND, UART_RX_IND
- wire segments 271 -> 308
- no-connect marks 2 -> 10
Other:
- moved on the sheet: C1, C10, C2, C3, C4, C5, C6, C7, C8, C9, C?, DL1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
